File: cart/kicad.real/kicad.kicad_pcb (KiCad board)
At the start: 4 copper layers, 100 x 64 mm, 23 parts, among them J1 Bus_TI994A_Cart, J2 Conn_01x06, U1 MCP1700-3302E_TO92, U2 S29GL01G-128MB-Flash, U3 GigaCart_CPLD_LC4064

Commit message: guess I never committed the working version...
Parts:
- removed !CS1, !CS2, !CS3, !CS4, !WE: ., Connectors:1pin
- added 35: ., Connectors:1pin, F.Cu at (163.2, 114.0)
- added C10: 1nF, Capacitors_SMD:C_0603_HandSoldering, B.Cu at (132.3, 104.0)
- added C3: 1nF, Capacitors_SMD:C_0603_HandSoldering, B.Cu at (149.2, 97.5)
- added C6: 1nF, Capacitors_SMD:C_0603_HandSoldering, B.Cu at (142.3, 82.0)
- added C8: 1nF, Capacitors_SMD:C_0603_HandSoldering, B.Cu at (140.1, 104.2)
- added C9: 1nF, Capacitors_SMD:C_0603_HandSoldering, B.Cu at (126.8, 98.0)
- added E1: ., Connectors:1pin, F.Cu at (165.5, 114.0)
- added E2: ., Connectors:1pin, F.Cu at (167.8, 114.0)
- added E3: ., Connectors:1pin, F.Cu at (170.0, 114.0)
- added E4: ., Connectors:1pin, F.Cu at (172.2, 114.0)
- R1: value 68^ -> 47^
- moved C7 4.37 mm to (132.0, 82.2)
- moved C1 0.71 mm to (131.5, 90.5)
- moved C4 0.71 mm to (142.5, 94.5)
- moved C2 0.50 mm to (138.1, 98.5)
Connections:
- J1 pad 21: Net-(J1-Pad21) -> TI_GSEL
- J1 pad 27: Net-(J1-Pad27) -> TI_GCLK
- U2 pad 14: +3V3 -> Net-(U2-Pad14)
- U2 pad 34: Net-(U2-Pad34) -> GND
- U3 pad 36: (no net) -> TI_GCLK
- U3 pad 44: Net-(J6-Pad1) -> TI_GSEL
- U3 pad 47: (no net) -> Net-(U2-Pad14)
- U3 pad 48: (no net) -> Net-(J6-Pad1)
- U3 pad 85: Net-(U2-Pad34) -> (no net)
Routing:
- net Net-(U2-Pad34): track 52.3 -> 0.00 mm
- net Net-(U2-Pad14): track 0.00 -> 41.2 mm, vias 0 -> 2
- net TI_GCLK: track 0.00 -> 30.4 mm, vias 0 -> 2
- net TI_GSEL: track 0.00 -> 28.2 mm, vias 0 -> 2
- net Net-(J6-Pad1): track 52.8 -> 37.0 mm
- net GND: track 72.6 -> 85.5 mm, vias 27 -> 32
- net Net-(J5-Pad1): track 49.4 -> 36.8 mm
- net Net-(J4-Pad1): track 46.0 -> 35.2 mm
- net Net-(J3-Pad1): track 42.6 -> 33.6 mm
- net +3V3: track 44.9 -> 53.9 mm, vias 21 -> 25
- net Net-(J7-Pad1): track 41.4 -> 35.3 mm
- net TI_ROM: track 43.1 -> 46.9 mm
- net TI_A4: track 36.6 -> 40.3 mm
- net TI_A5: track 36.5 -> 39.6 mm
- net TI_A6: track 36.6 -> 39.6 mm
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Other:
- board text added: "1"
- board text added: "2"
- board text added: "35"
- board text added: "36"
- board text added: "JTAG.Hdr 6 3v3 5 TDI 4 TCK 3 TMS 2 TDO 1 GND"
- board text removed: "JTAG.Hdr 1 GND 2 TDO 3 TMS 4 TCK 5 TDI 6 3v3"
